File: flowscript_demos/SimpleConsoleProgramExample.kicad_sch (KiCad schematic)
At the start: 12 parts

Commit message: Wow The whole day Was spent writting code I should have gone outside
Connections:
- new net: ADD1. (RES), fcs1., fcs3.
- new net: ADD1. (RES), fcs2., fcs3.
- new net: U2., U3., fa2.
